File: PCBs/KamiTrack.kicad_sch (KiCad schematic)
At the start: 63 parts, among them J1 Conn_01x02_Female, J2 Conn_01x04_Female, J3 Conn_01x02_Female, J4 Conn_01x08_Female, J5 Conn_01x02_Female, P1 USB_C_Plug_USB2.0, SW1 Option/FLASH Switch, SW2 Cali Switch, SW3 SW_SPDT MAIN POWER, U1 ME6211C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

Commit message: THIS IS VERY CURRECT JLCPCB_CORRECTION I SWEAR
Parts:
- D2, J3: JLCPCB_CORRECTION 0;0;0 -> 0;0;180
Changed lines of the file:
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@@
     )
     (property "LCSC" "C34499" (id 4) (at 41.91 59.69 0))
-    (property "JLCPCB_CORRECTION" "0;0;0" (id 5) (at 41.91 67.31 0))
+    (property "JLCPCB_CORRECTION" "0;0;180" (id 5) (at 41.91 67.31 0))
     (pin "1")
     (pin "2")
@@
     )
     (property "LCSC" "C173752" (id 4) (at 114.3 165.1 0))
-    (property "JLCPCB_CORRECTION" "0;0;0" (id 5) (at 115.57 158.75 0))
-    (pin "1")
-    (pin "2")
+    (property "JLCPCB_CORRECTION" "0;0;180" (id 5) (at 115.57 158.75 0))
+    (pin "1")
+    (pin "2")
