File: PCBs/KTracker.kicad_pcb (KiCad board)
At the start: 2 copper layers, 49.9 x 20.6 mm, 44 parts, among them J1 Conn_01x02_Female, J2 Conn_01x04_Female, P1 USB_C_Plug_USB2.0, SW1 Option/FLASH Switch, SW3 SW_SPDT MAIN POWER, U1 ME6211C, U2 TP4056, U6 ESP-12F, U7 CH340C, U9 MPU-9250

Commit message: add TS-1088R STEP
Routing:
- net VBAT: track 52.5 -> 32.4 mm, vias 4 -> 2
Other:
- board text added: "KTracker v0.5 SlimeVR Fullbody Tracker by Kamilake"
- board text removed: "KTracker v0.4 SlimeVR Fullbody Tracker"

Commit message: .
Parts:
- removed C1: 10uF, Capacitor_SMD:C_0402_1005Metric
- removed JST-MP: JST_GH_BM02B-GHS-TBT_1x02-1MP_P1.25mm_Vertical, Connector_JST:JST_GH_BM02B-GHS-TBT_1x02-1MP_P1.25mm_Vertical
- moved J2 18.2 mm to (136.5, 70.8), turned to 90 degrees
- moved R8 17.2 mm to (117.5, 74.4)
- moved R14 16.0 mm to (117.5, 70.4), turned to 180 degrees
- moved U2 15.1 mm to (122.6, 72.4)
- moved R4 14.2 mm to (117.5, 69.3), turned to 0 degrees
- moved R13 13.7 mm to (117.5, 71.4)
- moved R2 10.6 mm to (117.5, 73.4)
- moved C19 9.40 mm to (131.4, 65.4), turned to -90 degrees
- moved C20 9.07 mm to (133.5, 65.4), turned to -90 degrees
- moved R17 8.96 mm to (117.5, 72.4), turned to 180 degrees
- moved J1 6.90 mm to (139.0, 66.9)
- moved TP2 5.26 mm to (134.7, 74.0), turned to 90 degrees
- moved C10 4.19 mm to (134.1, 68.8), turned to 180 degrees
- moved C13 1.14 mm to (134.1, 67.8)
- moved TP1 0.92 mm to (138.7, 74.0)
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Routing:
- net GND: track 154.2 -> 95.1 mm, vias 46 -> 32
- net BATT+: track 70.0 -> 26.2 mm, vias 3 -> 0
- net +3V3: track 108.4 -> 67.0 mm, vias 13 -> 9
- net UART_ESP-: track 35.3 -> 10.3 mm, vias 2 -> 1
- net VBAT: track 32.4 -> 24.1 mm, vias 2 -> 0
- net VBUS: track 44.0 -> 36.2 mm, vias 6 -> 5
- net Net-(D2-Pad1): track 23.9 -> 18.3 mm
- net SDA: track 40.0 -> 45.2 mm, vias 4 -> 3
- net Net-(R2-Pad2): track 4.43 -> 0.00 mm, vias 2 -> 0
- net SCL: track 45.8 -> 41.7 mm, vias 4 -> 3
- net ADC: track 3.45 -> 0.00 mm
- net Net-(R4-Pad1): track 2.97 -> 0.00 mm, vias 2 -> 0
- net Net-(D1-Pad1): track 19.7 -> 17.1 mm
- net Net-(C7-Pad1): track 2.42 -> 0.00 mm
- net UART_ESP+: track 36.2 -> 38.4 mm
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Other:
- board size 49.9 x 20.6 mm -> 49.9 x 19.4 mm
- board text added: "-+"
- board text added: "Kamilake"
- board text added: "v0.5"
- board text removed: "+"
- board text removed: "-"
- board text removed: "Kamilake_"
- board text removed: "v0.5 es1"

Commit message: .
Parts:
- added C1: 10uF, Capacitor_SMD:C_0402_1005Metric, F.Cu at (134.1, 70.8)
- moved C13 2.03 mm to (134.1, 69.8)
Routing:
- net GND: track 95.1 -> 112.8 mm, vias 32 -> 26
- net VBUS: track 36.2 -> 51.1 mm, vias 5 -> 7
- net VBAT: track 24.1 -> 31.3 mm, vias 0 -> 1
- net BATT+: track 26.2 -> 28.2 mm, vias 0 -> 1

Commit message: !
Parts:
- moved R13 3.07 mm to (117.5, 74.4)
- moved R14 3.07 mm to (117.5, 73.4)
- moved G*** 3.05 mm to (125.6, 65.1)
- moved R2 2.03 mm to (117.5, 71.4)
- moved R17 2.03 mm to (117.5, 70.4)
- moved R8 2.03 mm to (117.5, 72.4)
- moved C19 0.27 mm to (131.6, 65.6)
- moved C20 0.27 mm to (133.6, 65.6)
Routing:
- net GND: track 112.8 -> 163.0 mm, vias 26 -> 35
- net +3V3: track 67.0 -> 116.1 mm, vias 9 -> 14
- net BATT+: track 28.2 -> 67.4 mm, vias 1 -> 4
- net UART_ESP-: track 10.3 -> 35.6 mm, vias 1 -> 2
- net Net-(R8-Pad2): track 0.00 -> 17.9 mm, vias 0 -> 2
- net ADC: track 0.00 -> 16.4 mm, vias 0 -> 2
- net Net-(R2-Pad2): track 0.00 -> 15.7 mm, vias 0 -> 2
- net Net-(R17-Pad2): track 0.00 -> 10.6 mm, vias 0 -> 2
- net Net-(R4-Pad1): track 0.00 -> 5.41 mm, vias 0 -> 2
- net Net-(C7-Pad1): track 0.00 -> 1.22 mm
- net VBUS: track 51.1 -> 50.3 mm
- net Net-(P1-PadA7): track 7.07 -> 7.89 mm
- net Net-(D1-Pad1): track 17.1 -> 16.3 mm
- net Net-(D1-Pad2): track 2.46 -> 1.93 mm
- net SDA: vias 3 -> 2
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Other:
- board text added: "4.2v/SDA/SCL/GND"
- board text added: "B+/B-"
- board text added: "MPU6500"
- board text added: "v5"
- board text removed: "v0.5"

Commit message: .
Routing:
- net Net-(P1-PadA7): track 7.89 -> 7.08 mm
- net GND: vias 35 -> 45
Other:
- board text removed: "SlimeVR"
Changed lines of the file:
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@@
     (effects (font (size 1 1) (thickness 0.15)))
   )
-  (gr_text "-+" (at 136.779 74.803) (layer "F.SilkS")
+  (gr_text "-+" (at 136.7536 74.6252) (layer "F.SilkS")
     (effects (font (size 1 1) (thickness 0.2)))
   )
   (gr_text "Kamilake" (at 130.048 74.295) (layer "F.SilkS")
-    (effects (font (size 1 1) (thickness 0.15)))
-  )
-  (gr_text "SlimeVR" (at 125.222 77.724) (layer "F.SilkS")
     (effects (font (size 1 1) (thickness 0.15)))
   )
@@
   (segment (start 130.8328 61.6484) (end 131.116 61.9316) (width 0.2) (layer "F.Cu") (net 1))
   (segment (start 119.905 69.988) (end 120.424 69.469) (width 0.4) (layer "F.Cu") (net 1))
-  (segment (start 133.632 70.8406) (end 133.632 66.51) (width 0.4) (layer "F.Cu") (net 1))
+  (segment (start 133.632 70.8406) (end 133.632 67.7138) (width 0.4) (layer "F.Cu") (net 1))
   (segment (start 112.395 60.419) (end 112.395 62.485) (width 0.4) (layer "F.Cu") (net 1))
   (segment (start 120.1166 61.468) (end 121.2748 61.468) (width 0.2) (layer "F.Cu") (net 1))
@@
   (segment (start 133.477 66.5836) (end 131.445 66.5836) (width 0.4) (layer "F.Cu") (net 1))
   (segment (start 132.29 72.77) (end 132.29 72.4) (width 0.4) (layer "F.Cu") (net 1))
+  (segment (start 133.632 67.7138) (end 133.632 66.51) (width 0.4) (layer "F.Cu") (net 1))
   (segment (start 138.686 56.8366) (end 138.686 61.0166) (width 0.2) (layer "F.Cu") (net 1))
   (via (at 98.933 67.564) (size 0.4) (drill 0.3) (layers "F.Cu" "B.Cu") (free) (net 1))
@@
   (via (at 98.933 63.5) (size 0.4) (drill 0.3) (layers "F.Cu" "B.Cu") (free) (net 1))
   (via (at 125.5014 65.659) (size 0.4) (drill 0.3) (layers "F.Cu" "B.Cu") (free) (net 1))
+  (via (at 107.2642 61.5442) (size 0.4) (drill 0.3) (layers "F.Cu" "B.Cu") (free) (net 1))
   (via (at 136.017 59.436) (size 0.4) (drill 0.3) (layers "F.Cu" "B.Cu") (free) (net 1))
   (via (at 98.933 70.612) (size 0.4) (drill 0.3) (layers "F.Cu" "B.Cu") (free) (net 1))
+  (via (at 127.4064 73.6854) (size 0.4) (drill 0.3) (layers "F.Cu" "B.Cu") (free) (net 1))
+  (via (at 109.8042 62.5094) (size 0.4) (drill 0.3) (layers "F.Cu" "B.Cu") (free) (net 1))
+  (via (at 138.9888 64.4652) (size 0.4) (drill 0.3) (layers "F.Cu" "B.Cu") (free) (net 1))
   (via (at 137.16 72.3646) (size 0.8) (drill 0.4) (layers "F.Cu" "B.Cu") (net 1))
   (via (at 98.933 62.484) (size 0.4) (drill 0.3) (layers "F.Cu" "B.Cu") (free) (net 1))
@@
   (via (at 112.395 64.3128) (size 0.4) (drill 0.3) (layers "F.Cu" "B.Cu") (net 1))
   (via (at 112.395 70.866) (size 0.4) (drill 0.3) (layers "F.Cu" "B.Cu") (net 1))
+  (via (at 109.8042 65.3542) (size 0.4) (drill 0.3) (layers "F.Cu" "B.Cu") (free) (net 1))
   (via (at 98.933 71.628) (size 0.4) (drill 0.3) (layers "F.Cu" "B.Cu") (free) (net 1))
   (via (at 120.015 69.469) (size 0.4) (drill 0.3) (layers "F.Cu" "B.Cu") (net 1))
@@
   (via (at 98.933 64.516) (size 0.4) (drill 0.3) (layers "F.Cu" "B.Cu") (free) (net 1))
   (via (at 98.933 65.532) (size 0.4) (drill 0.3) (layers "F.Cu" "B.Cu") (free) (net 1))
+  (via (at 109.7534 68.9102) (size 0.4) (drill 0.3) (layers "F.Cu" "B.Cu") (free) (net 1))
   (via (at 118.5926 69.469) (size 0.4) (drill 0.3) (layers "F.Cu" "B.Cu") (net 1))
   (via (at 130.4544 64.0588) (size 0.4) (drill 0.3) (layers "F.Cu" "B.Cu") (net 1))
   (via (at 128.0272 69.4395) (size 0.8) (drill 0.4) (layers "F.Cu" "B.Cu") (net 1))
   (via (at 127.6858 59.2836) (size 0.4) (drill 0.3) (layers "F.Cu" "B.Cu") (net 1))
+  (via (at 129.6162 73.6346) (size 0.4) (drill 0.3) (layers "F.Cu" "B.Cu") (free) (net 1))
   (via (at 136.5504 74.7776) (size 0.4) (drill 0.3) (layers "F.Cu" "B.Cu") (free) (net 1))
   (via (at 132.207 70.805) (size 0.8) (drill 0.4) (layers "F.Cu" "B.Cu") (net 1))
@@
   (via (at 112.395 69.469) (size 0.4) (drill 0.3) (layers "F.Cu" "B.Cu") (net 1))
   (via (at 98.933 61.468) (size 0.4) (drill 0.3) (layers "F.Cu" "B.Cu") (free) (net 1))
+  (via (at 133.632 67.7138) (size 0.4) (drill 0.3) (layers "F.Cu" "B.Cu") (net 1))
   (via (at 120.8871 64.3128) (size 0.4) (drill 0.3) (layers "F.Cu" "B.Cu") (net 1))
+  (via (at 126.0544 61.0166) (size 0.4) (drill 0.3) (layers "F.Cu" "B.Cu") (net 1))
+  (via (at 102.616 61.4934) (size 0.4) (drill 0.3) (layers "F.Cu" "B.Cu") (free) (net 1))
   (via (at 98.933 66.548) (size 0.4) (drill 0.3) (layers "F.Cu" "B.Cu") (free) (net 1))
   (via (at 119.5324 61.7728) (size 0.4) (drill 0.3) (layers "F.Cu" "B.Cu") (net 1))
@@
   (segment (start 98.933 71.628) (end 98.933 60.452) (width 0.3) (layer "B.Cu") (net 1))
   (segment (start 138.9518 66.9196) (end 138.9518 67.131338) (width 0.5) (layer "B.Cu") (net 1))
-  (segment (start 130.046 61.0166) (end 120.2886 61.0166) (width 0.2) (layer "B.Cu") (net 1))
+  (segment (start 130.046 61.0166) (end 126.0544 61.0166) (width 0.2) (layer "B.Cu") (net 1))
   (segment (start 128.1295 69.4395) (end 128.0272 69.4395) (width 0.5) (layer "B.Cu") (net 1))
   (segment (start 134.747 74.041) (end 135.4836 74.041) (width 0.4) (layer "B.Cu") (net 1))
@@
   (segment (start 130.046 61.0166) (end 128.313 59.2836) (width 0.2) (layer "B.Cu") (net 1))
   (segment (start 130.046 61.0166) (end 130.046 56.8366) (width 0.25) (layer "B.Cu") (net 1))
+  (segment (start 126.0544 61.0166) (end 120.2886 61.0166) (width 0.2) (layer "B.Cu") (net 1))
   (segment (start 135.4836 74.041) (end 137.16 72.3646) (width 0.4) (layer "B.Cu") (net 1))
   (segment (start 131.2136 64.818) (end 136.488 64.818) (width 0.25) (layer "B.Cu") (net 1))
@@
   (segment (start 135.3058 63.627) (end 135.3058 63.0936) (width 0.3) (layer "B.Cu") (net 13))
   (segment (start 108.585 58.928) (end 108.585 60.4012) (width 0.2) (layer "B.Cu") (net 13))
-  (segment (start 124.34832 62.42312) (end 124.34832 62.44852) (width 0.3) (layer "B.Cu") (net 13))
   (segment (start 134.6708 64.262) (end 135.3058 63.627) (width 0.3) (layer "B.Cu") (net 13))
   (segment (start 118.4148 68.0212) (end 121.3866 68.0212) (width 0.2) (layer "B.Cu") (net 13))
-  (segment (start 130.556 62.4078) (end 130.406202 62.4078) (width 0.3) (layer "B.Cu") (net 13))
   (segment (start 121.3866 68.0212) (end 125.3635 68.0212) (width 0.2) (layer "B.Cu") (net 13))
   (segment (start 128.397 73.5971) (end 128.826711 73.167389) (width 0.4) (layer "B.Cu") (net 13))
@@
   (segment (start 129.3114 62.97262) (end 128.04658 62.97262) (width 0.3) (layer "F.Cu") (net 40))
   (segment (start 134.116 62.861976) (end 134.116 61.9316) (width 0.2) (layer "F.Cu") (net 40))
-  (segment (start 128.0272 62.992) (end 128.8288 62.992) (width 0.2) (layer "F.Cu") (net 40))
   (segment (start 133.991819 62.986157) (end 134.116 62.861976) (width 0.2) (layer "F.Cu") (net 40))
   (via (at 129.3114 62.97262) (size 0.4) (drill 0.3) (layers "F.Cu" "B.Cu") (net 40))
   (via (at 133.991819 62.986157) (size 0.4) (drill 0.3) (layers "F.Cu" "B.Cu") (net 40))
   (segment (start 133.991819 62.986157) (end 129.324937 62.986157) (width 0.3) (layer "B.Cu") (net 40))
-  (segment (start 133.985976 62.992) (end 133.991819 62.986157) (width 0.2) (layer "B.Cu") (net 40))
   (segment (start 129.324937 62.986157) (end 129.3114 62.97262) (width 0.3) (layer "B.Cu") (net 40))
   (segment (start 134.616 61.9316) (end 134.616 63.239252) (width 0.2) (layer "F.Cu") (net 42))

Commit message: ..!
Routing:
- net GND: vias 45 -> 47
Other:
- board text added: "2022-09-04 KTracker v5"
- board text added: "KTracker v5 SlimeVR Fullbody Tracker by Kamilake"
- board text added: "https://github.com/Kamilake/KTracker-SlimeVR-PCB"
- board text removed: "KTracker v0.5 SlimeVR Fullbody Tracker by Kamilake"
Changed lines of the file:
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@@
     (property "Sheetname" "")
     (attr through_hole)
-    (fp_text reference "J1" (at 1 2.55 90) (layer "B.SilkS")
+    (fp_text reference "J1" (at 5.1402 -5.5742 90) (layer "B.Fab")
       (effects (font (size 1 1) (thickness 0.15)) (justify mirror))
     )
@@
   (gr_line (start 140.081 75.184) (end 90.17 75.184) (layer "Edge.Cuts") (width 0.05))
   (gr_line (start 90.17 75.184) (end 90.17 55.753) (layer "Edge.Cuts") (width 0.05))
+  (gr_text "https://github.com/Kamilake/KTracker-SlimeVR-PCB" (at 107.9246 58.547) (layer "B.SilkS")
+    (effects (font (size 0.8 0.8) (thickness 0.13)) (justify mirror))
+  )
   (gr_text "4.2v/SDA/SCL/GND" (at 135.5344 59.7662 270) (layer "B.SilkS")
     (effects (font (size 0.7 0.5) (thickness 0.1)) (justify mirror))
@@
     (effects (font (size 0.7 0.5) (thickness 0.1)) (justify mirror))
   )
+  (gr_text "2022-09-04 KTracker v5" (at 100.2792 56.9722) (layer "B.SilkS")
+    (effects (font (size 0.9 0.9) (thickness 0.14)) (justify mirror))
+  )
   (gr_text "-+" (at 138.7348 72.4408 180) (layer "B.SilkS")
     (effects (font (size 1 1) (thickness 0.2)) (justify mirror))
   )
-  (gr_text "KTracker v0.5 SlimeVR Fullbody Tracker by Kamilake" (at 114.04 79.94) (layer "F.SilkS")
+  (gr_text "KTracker v5 SlimeVR Fullbody Tracker by Kamilake" (at 114.04 79.94) (layer "F.SilkS")
     (effects (font (size 1 1) (thickness 0.15)))
   )
@@
     (effects (font (size 0.7 0.7) (thickness 0.12)))
   )
-  (dimension (type aligned) (layer "F.Fab")
-    (pts (xy 89.789 106.299) (xy 89.789 85.725))
-    (height -3.6068)
-    (gr_text "20.5740 mm" (at 85.0322 96.012 90) (layer "F.Fab")
-      (effects (font (size 1 1) (thickness 0.15)))
-    )
-    (format (units 3) (units_format 1) (precision 4))
-    (style (thickness 0.1) (arrow_length 1.27) (text_position_mode 0) (extension_height 0.58642) (extension_offset 0.5) keep_text_aligned)
-  )
-  (dimension (type aligned) (layer "F.Fab")
-    (pts (xy 89.789 91.9734) (xy 139.7 91.9734))
-    (height -8.6614)
-    (gr_text "49.9110 mm" (at 114.7445 82.162) (layer "F.Fab")
-      (effects (font (size 1 1) (thickness 0.15)))
-    )
-    (format (units 3) (units_format 1) (precision 4))
-    (style (thickness 0.1) (arrow_length 1.27) (text_position_mode 0) (extension_height 0.58642) (extension_offset 0.5) keep_text_aligned)
-  )
   (segment (start 127.6838 58.8772) (end 127.6838 59.2816) (width 0.5) (layer "F.Cu") (net 1))
   (segment (start 120.499 64.3142) (end 120.8857 64.3142) (width 0.2) (layer "F.Cu") (net 1))
@@
   (via (at 127.4064 73.6854) (size 0.4) (drill 0.3) (layers "F.Cu" "B.Cu") (free) (net 1))
   (via (at 109.8042 62.5094) (size 0.4) (drill 0.3) (layers "F.Cu" "B.Cu") (free) (net 1))
+  (via (at 114.8334 68.0212) (size 0.4) (drill 0.3) (layers "F.Cu" "B.Cu") (free) (net 1))
   (via (at 138.9888 64.4652) (size 0.4) (drill 0.3) (layers "F.Cu" "B.Cu") (free) (net 1))
   (via (at 137.16 72.3646) (size 0.8) (drill 0.4) (layers "F.Cu" "B.Cu") (net 1))
+  (via (at 115.6462 72.9234) (size 0.4) (drill 0.3) (layers "F.Cu" "B.Cu") (free) (net 1))
   (via (at 98.933 62.484) (size 0.4) (drill 0.3) (layers "F.Cu" "B.Cu") (free) (net 1))
   (via (at 139.446 71.628) (size 0.4) (drill 0.3) (layers "F.Cu" "B.Cu") (free) (net 1))

Commit message: .
Parts:
- added G***: LOGO, kamilib:FineMotion_18mm, B.Cu at (116.1, 72.9)
Other:
- board text added: "2022-09-24 KTracker v5"
- board text added: "v5a"
- board text removed: "2022-09-04 KTracker v5"
- board text removed: "v5"

Commit message: .
Parts:
- moved G*** 100.0 mm to (198.8, 68.2)
Changed lines of the file:
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@@
   )
   (footprint "kamilib:sleepy300dpi" (layer "B.Cu")
-    (at 98.84 68.16 180)
+    (at 198.84 68.16 180)
     (attr through_hole)
     (fp_text reference "G***" (at 0 0) (layer "B.SilkS") hide
