File: AUX_PCBs/KTracker_AUX.kicad_sch (KiCad schematic)
At the start: 11 parts, among them J2 Conn_01x04_Female, U1 ME6211C, U9 MPU-9250

Commit message: .
Connections:
- net +3V3: now also U9.9 (AD0/MISO)
- net GND: no longer U9.9 (AD0/MISO)
- net AUX_SCL: no longer names the net of U9.7 (AUX_SCL)
- net AUX_SDA: no longer names the net of U9.21 (AUX_SDA)
- no-connect marks 9 -> 5
Changed lines of the file:
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@@
     (comment 2 "Compatible with github.com/SlimeVR/SlimeVR-Tracker-ESP")
   )
-  (junction (at 40.64 143.51) (diameter 0) (color 0 0 0 0)
-  )
-  (junction (at 64.77 157.48) (diameter 0) (color 0 0 0 0)
-  )
-  (junction (at 76.2 143.51) (diameter 0) (color 0 0 0 0)
-  )
   (junction (at 236.22 21.59) (diameter 0) (color 0 0 0 0)
   )
@@
   (junction (at 224.79 21.59) (diameter 0) (color 0 0 0 0)
   )
-  (junction (at 44.45 158.75) (diameter 0) (color 0 0 0 0)
-  )
-  (junction (at 50.8 143.51) (diameter 0) (color 0 0 0 0)
-  )
   (junction (at 35.56 162.56) (diameter 0) (color 0 0 0 0)
   )
@@
   (junction (at 241.3 21.59) (diameter 0) (color 0 0 0 0)
   )
-  (junction (at 44.45 143.51) (diameter 0) (color 0 0 0 0)
+  (junction (at 210.82 21.59) (diameter 0) (color 0 0 0 0)
+  )
+  (junction (at 34.29 151.13) (diameter 0) (color 0 0 0 0)
   )
   (junction (at 40.64 151.13) (diameter 0) (color 0 0 0 0)
@@
   )
   (junction (at 43.18 170.18) (diameter 0) (color 0 0 0 0)
-  )
-  (junction (at 210.82 53.34) (diameter 0) (color 0 0 0 0)
   )
   (junction (at 238.76 72.39) (diameter 0) (color 0 0 0 0)
@@
   (no_connect (at 256.54 40.64))
   (no_connect (at 74.93 146.05))
-  (no_connect (at 76.2 148.59))
+  (no_connect (at 256.54 45.72))
   (no_connect (at 256.54 55.88))
-  (no_connect (at 50.8 151.13))
-  (no_connect (at 76.2 156.21))
-  (no_connect (at 44.45 144.78))
-  (no_connect (at 44.45 152.4))
-  (no_connect (at 35.56 143.51))
-  (bus_entry (at -675.64 227.33) (size 2.54 2.54)
+  (no_connect (at 256.54 48.26))
+  (wire (pts (xy 210.82 21.59) (xy 210.82 43.18))
     (stroke (width 0) (type default) (color 0 0 0 0))
   )
@@
     (stroke (width 0) (type default) (color 0 0 0 0))
   )
-  (wire (pts (xy 35.56 143.51) (xy 40.64 143.51))
-    (stroke (width 0) (type default) (color 0 0 0 0))
-  )
   (polyline (pts (xy 50.8 195.58) (xy 50.8 175.26))
     (stroke (width 0) (type default) (color 0 0 0 0))
@@
     (stroke (width 0) (type default) (color 0 0 0 0))
   )
-  (wire (pts (xy 64.77 153.67) (xy 64.77 157.48))
-    (stroke (width 0) (type default) (color 0 0 0 0))
-  )
   (wire (pts (xy 189.23 54.61) (xy 193.04 54.61))
     (stroke (width 0) (type default) (color 0 0 0 0))
@@
     (stroke (width 0) (type default) (color 0 0 0 0))
   )
-  (wire (pts (xy 50.8 143.51) (xy 54.61 143.51))
-    (stroke (width 0) (type default) (color 0 0 0 0))
-  )
-  (wire (pts (xy 44.45 143.51) (xy 50.8 143.51))
-    (stroke (width 0) (type default) (color 0 0 0 0))
-  )
-  (wire (pts (xy 80.01 143.51) (xy 76.2 143.51))
+  (wire (pts (xy 74.93 143.51) (xy 80.01 143.51))
     (stroke (width 0) (type default) (color 0 0 0 0))
   )
@@
     (stroke (width 0) (type default) (color 0 0 0 0))
   )
-  (wire (pts (xy 76.2 156.21) (xy 76.2 157.48))
-    (stroke (width 0) (type default) (color 0 0 0 0))
-  )
-  (wire (pts (xy 76.2 143.51) (xy 74.93 143.51))
-    (stroke (width 0) (type default) (color 0 0 0 0))
-  )
-  (wire (pts (xy 30.48 151.13) (xy 40.64 151.13))
+  (wire (pts (xy 34.29 151.13) (xy 40.64 151.13))
+    (stroke (width 0) (type default) (color 0 0 0 0))
+  )
+  (wire (pts (xy 30.48 151.13) (xy 34.29 151.13))
     (stroke (width 0) (type default) (color 0 0 0 0))
   )
@@
     (stroke (width 0) (type default) (color 0 0 0 0))
   )
-  (wire (pts (xy 44.45 152.4) (xy 44.45 158.75))
-    (stroke (width 0) (type default) (color 0 0 0 0))
-  )
   (wire (pts (xy 31.75 185.42) (xy 36.83 185.42))
     (stroke (width 0) (type default) (color 0 0 0 0))
   )
-  (wire (pts (xy 76.2 148.59) (xy 76.2 143.51))
+  (wire (pts (xy 210.82 21.59) (xy 217.17 21.59))
     (stroke (width 0) (type default) (color 0 0 0 0))
   )
@@
     (stroke (width 0) (type default) (color 0 0 0 0))
   )
-  (wire (pts (xy 44.45 144.78) (xy 44.45 143.51))
-    (stroke (width 0) (type default) (color 0 0 0 0))
-  )
-  (wire (pts (xy 50.8 151.13) (xy 50.8 143.51))
-    (stroke (width 0) (type default) (color 0 0 0 0))
-  )
   (polyline (pts (xy 182.88 15.24) (xy 280.67 15.24))
     (stroke (width 0) (type default) (color 0 0 0 0))
@@
     (stroke (width 0) (type default) (color 0 0 0 0))
   )
-  (wire (pts (xy 40.64 158.75) (xy 44.45 158.75))
-    (stroke (width 0) (type default) (color 0 0 0 0))
-  )
-  (wire (pts (xy 64.77 157.48) (xy 64.77 158.75))
-    (stroke (width 0) (type default) (color 0 0 0 0))
-  )
-  (wire (pts (xy 40.64 143.51) (xy 44.45 143.51))
+  (wire (pts (xy 40.64 158.75) (xy 64.77 158.75))
+    (stroke (width 0) (type default) (color 0 0 0 0))
+  )
+  (wire (pts (xy 64.77 153.67) (xy 64.77 158.75))
+    (stroke (width 0) (type default) (color 0 0 0 0))
+  )
+  (wire (pts (xy 40.64 143.51) (xy 54.61 143.51))
     (stroke (width 0) (type default) (color 0 0 0 0))
   )
@@
     (stroke (width 0) (type default) (color 0 0 0 0))
   )
-  (wire (pts (xy 260.35 48.26) (xy 256.54 48.26))
-    (stroke (width 0) (type default) (color 0 0 0 0))
-  )
   (wire (pts (xy 200.66 46.99) (xy 200.66 52.07))
     (stroke (width 0) (type default) (color 0 0 0 0))
@@
     (stroke (width 0) (type default) (color 0 0 0 0))
   )
-  (wire (pts (xy 210.82 43.18) (xy 210.82 53.34))
-    (stroke (width 0) (type default) (color 0 0 0 0))
-  )
   (wire (pts (xy 260.35 53.34) (xy 256.54 53.34))
     (stroke (width 0) (type default) (color 0 0 0 0))
@@
     (stroke (width 0) (type default) (color 0 0 0 0))
   )
-  (wire (pts (xy 256.54 45.72) (xy 260.35 45.72))
-    (stroke (width 0) (type default) (color 0 0 0 0))
-  )
   (wire (pts (xy 193.04 21.59) (xy 200.66 21.59))
     (stroke (width 0) (type default) (color 0 0 0 0))
@@
     (stroke (width 0) (type default) (color 0 0 0 0))
   )
-  (wire (pts (xy 76.2 157.48) (xy 64.77 157.48))
-    (stroke (width 0) (type default) (color 0 0 0 0))
-  )
   (wire (pts (xy 238.76 72.39) (xy 238.76 71.12))
     (stroke (width 0) (type default) (color 0 0 0 0))
@@
     (stroke (width 0) (type default) (color 0 0 0 0))
   )
-  (wire (pts (xy 200.66 21.59) (xy 217.17 21.59))
+  (wire (pts (xy 200.66 21.59) (xy 210.82 21.59))
     (stroke (width 0) (type default) (color 0 0 0 0))
   )
@@
   )
   (wire (pts (xy 217.17 48.26) (xy 217.17 21.59))
-    (stroke (width 0) (type default) (color 0 0 0 0))
-  )
-  (wire (pts (xy 44.45 158.75) (xy 64.77 158.75))
     (stroke (width 0) (type default) (color 0 0 0 0))
   )
@@
     )
   )
-  (global_label "AUX_SDA" (shape output) (at 260.35 45.72 0) (fields_autoplaced)
-    (effects (font (size 1.27 1.27)) (justify left))
-    (property "Intersheet References" "${INTERSHEET_REFS}" (id 0) (at 7.62 -82.55 0)
-      (effects (font (size 1.27 1.27)) hide)
-    )
-  )
   (global_label "SCL" (shape input) (at 189.23 54.61 180) (fields_autoplaced)
     (effects (font (size 1.27 1.27)) (justify right))
     (property "Intersheet References" "${INTERSHEET_REFS}" (id 0) (at 7.62 -81.28 0)
-      (effects (font (size 1.27 1.27)) hide)
-    )
-  )
-  (global_label "AUX_SCL" (shape output) (at 260.35 48.26 0) (fields_autoplaced)
-    (effects (font (size 1.27 1.27)) (justify left))
-    (property "Intersheet References" "${INTERSHEET_REFS}" (id 0) (at 7.62 -82.55 0)
       (effects (font (size 1.27 1.27)) hide)
     )
@@
     )
     (property "Datasheet" "" (id 3) (at 52.07 170.18 0)
+      (effects (font (size 1.27 1.27)) hide)
+    )
+    (pin "1")
+  )
+  (symbol (lib_id "power:PWR_FLAG") (at 34.29 151.13 0) (unit 1)
+    (in_bom yes) (on_board yes) (fields_autoplaced)
+    (property "Reference" "#FLG0101" (id 0) (at 34.29 149.225 0)
+      (effects (font (size 1.27 1.27)) hide)
+    )
+    (property "Value" "PWR_FLAG" (id 1) (at 34.29 147.5255 0))
+    (property "Footprint" "" (id 2) (at 34.29 151.13 0)
+      (effects (font (size 1.27 1.27)) hide)
+    )
+    (property "Datasheet" "~" (id 3) (at 34.29 151.13 0)
       (effects (font (size 1.27 1.27)) hide)
     )
@@
   )
   (symbol_instances
+    (path "/20514691-7a9b-4cbe-8bec-ec3f68a1f041"
+      (reference "#FLG0101") (unit 1) (value "PWR_FLAG") (footprint "")
+    )
     (path "/00000000-0000-0000-0000-000061ae078e"
       (reference "#PWR02") (unit 1) (value "+3.3V") (footprint "")
